Commit message: feat(gsmini): create new sensor

File: tactile_gym/assets/robot_assets/gelsight_mini/standard_gelsight_mini/gelsight_mini_asmb/urdf/gelsight_mini_asmb.urdf (robot description, URDF)
Before this commit: robot digit_asmb, 2 links, 1 joints
Links:
- removed link digit_body
- removed link digit_core
- added link gsmini_body, mass 0.0077837104153161; collision mesh filename=package://gelsight_mini_asmb/meshes/gsmini_body.STL; visual mesh filename=package://gelsight_mini_asmb/meshes/gsmini_body.STL
- added link gsmini_core, mass 0.00130411151086353; collision mesh filename=package://gelsight_mini_asmb/meshes/gsmini_core.STL; visual mesh filename=package://gelsight_mini_asmb/meshes/gsmini_core.STL
Joints:
- removed joint digit_body_core_link
- added joint gsmini_body_core_link: type fixed, parent digit_body, child digit_core, origin xyz=-0.00151521951809463 -1.36251105150219E-05 -0.00415 rpy=-3.14159265358979 0 1.5707963267949, axis 0 0 0

Commit message: fix(urdf): fix gelsight mini asmb

File: tactile_gym/assets/robot_assets/gelsight_mini/standard_gelsight_mini/gelsight_mini_asmb/urdf/gelsight_mini_asmb.urdf (robot description, URDF)
Before this commit: robot gsmini_asmb, 2 links, 1 joints
Joints:
- joint gsmini_body_core_link: child digit_core -> gsmini_core; parent digit_body -> gsmini_body
