Commit message: fix(gsmini): position and rotation for ur5

File: tactile_gym/assets/robot_assets/ur5/gelsight_mini/ur5_with_standard_gelsight_mini.urdf (robot description, URDF)
Before this commit: robot universal_robot, 12 links, 11 joints
Joints:
- joint tcp_joint: origin xyz=0.0007 0.0 0.040 rpy=0 0 0 -> xyz=0.0007 0.0 0.0215 rpy=0 0 0
