Commit message: fix(gsmini): create hollow assembly and fix names

File: tactile_gym/assets/robot_assets/franka_panda/gelsight_mini/franka_panda_with_standard_gelsight_mini.urdf (robot description, URDF)
Before this commit: robot panda, 13 links, 12 joints
Links:
- removed link gsmini_body_link
- removed link gsmini_tip_link
- added link gelsight_mini_body_link, mass 0.0077837104153161; collision mesh filename=../gelsight_mini/standard_gelsight_mini/gelsight_mini_asmb/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; visual mesh filename=../gelsight_mini/standard_gelsight_mini/gelsight_mini_asmb/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
- added link gelsight_mini_tip_link, mass 0.00130411151086353; collision mesh filename=../gelsight_mini/standard_gelsight_mini/gelsight_mini_asmb/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; visual mesh filename=../gelsight_mini/standard_gelsight_mini/gelsight_mini_asmb_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 scale=1.0 1.0 1.0
Joints:
- removed joint dgsmini_ee_joint
- removed joint gsmini_tip_to_body
- added joint dgelsight_mini_ee_joint: type fixed, parent ee_link, child gelsight_mini_body_link, origin xyz=0.0 0.0 0.0 rpy=0.0 0.0 -1.57
- added joint gelsight_mini_tip_to_body: type fixed, parent gelsight_mini_body_link, child gelsight_mini_tip_link, origin xyz=-0.00151521951809463 -1.36251105150219E-05 -0.00415 rpy=-3.14159265358979 0 1.5707963267949, axis 0 0 0
- joint tcp_joint: parent gsmini_body_link -> gelsight_mini_body_link

File: tactile_gym/assets/robot_assets/gelsight_mini/standard_gelsight_mini/gelsight_mini_asmb_hollow/urdf/gelsight_mini_asmb_hollow.urdf (robot description, URDF)
Before this commit: robot gelsight_mini_asmb, 2 links, 1 joints
Links:
- link gelsight_mini_body: geometry collision mesh filename=package://gelsight_mini_asmb_hollow/meshes/gelsight_mini_bo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; visual mesh filename=package://gelsight_mini_asmb_hollow/meshes/gelsight_mini_bo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
- link gelsight_mini_core: mass 0.00130411151086353 -> 1.15850364457513E-05; geometry collision mesh filename=package://gelsight_mini_asmb_hollow/meshes/gelsight_mini_co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; visual mesh filename=package://gelsight_mini_asmb_hollow/meshes/gelsight_mini_co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

File: tactile_gym/assets/robot_assets/kuka_iiwa/gelsight_mini/kuka_iiwa_with_standard_gelsight_mini.urdf (robot description, URDF)
Before this commit: robot lbr_iiwa, 13 links, 12 joints
Links:
- removed link gsmini_body_link
- removed link gsmini_tip_link
- added link gelsight_mini_body_link, mass 0.0077837104153161; collision mesh filename=../gelsight_mini/standard_gelsight_mini/gelsight_mini_asmb/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; visual mesh filename=../gelsight_mini/standard_gelsight_mini/gelsight_mini_asmb/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
- added link gelsight_mini_tip_link, mass 0.00130411151086353; collision mesh filename=../gelsight_mini/standard_gelsight_mini/gelsight_mini_asmb/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; visual mesh filename=../gelsight_mini/standard_gelsight_mini/gelsight_mini_asmb_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 scale=1.0 1.0 1.0
Joints:
- removed joint gsmini_ee_joint
- removed joint gsmini_tip_to_body
- added joint gelsight_mini_ee_joint: type fixed, parent ee_link, child gelsight_mini_body_link, origin xyz=0.0 0.0 0.0 rpy=-3.14 0.0 3.14
- added joint gelsight_mini_tip_to_body: type fixed, parent gelsight_mini_body_link, child gelsight_mini_tip_link, origin xyz=-0.00151521951809463 -1.36251105150219E-05 -0.00415 rpy=-3.14159265358979 0 1.5707963267949, axis 0 0 0
- joint tcp_joint: parent gsmini_body_link -> gelsight_mini_body_link

Commit message: fix(gsmini): fix meshes and support on franka panda

File: tactile_gym/assets/robot_assets/franka_panda/gelsight_mini/franka_panda_with_standard_gelsight_mini.urdf (robot description, URDF)
Before this commit: robot panda, 13 links, 12 joints
Joints:
- removed joint dgelsight_mini_ee_joint
- added joint gelsight_mini_ee_joint: type fixed, parent ee_link, child gelsight_mini_body_link, origin xyz=0.0 0.0 0.0 rpy=0.0 0.0 -1.57

Commit message: fix(gsmini): fix position and rotation for panda and kuka

File: tactile_gym/assets/robot_assets/franka_panda/gelsight_mini/franka_panda_with_standard_gelsight_mini.urdf (robot description, URDF)
Before this commit: robot panda, 13 links, 12 joints
Joints:
- joint tcp_joint: origin xyz=0.0007 0.0 0.040 rpy=0 0 0 -> xyz=0.0007 0.0 0.0215 rpy=0 0 0

File: tactile_gym/assets/robot_assets/kuka_iiwa/gelsight_mini/kuka_iiwa_with_standard_gelsight_mini.urdf (robot description, URDF)
Before this commit: robot lbr_iiwa, 13 links, 12 joints
Joints:
- joint tcp_joint: origin xyz=0.0007 0.0 0.040 rpy=0 0 0 -> xyz=0.0007 0.0 0.0195 rpy=0 0 0

Commit message: refactor(gsmini): colors with franka panda

File: tactile_gym/assets/robot_assets/franka_panda/gelsight_mini/franka_panda_with_standard_gelsight_mini.urdf (robot description, URDF)
Before this commit: robot panda, 13 links, 12 joints
Links:
- link gelsight_mini_tip_link: geometry collision mesh filename=../gelsight_mini/standard_gelsight_mini/gelsight_mini_asmb/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; visual mesh filename=../gelsight_mini/standard_gelsight_mini/gelsight_mini_asmb_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
